File: kicad/thermo.sch (KiCad schematic (older format))
At the start: 55 parts, among them P1 CONN_VREF, P10 CONN_STM32F030_11_20, P11 CONN_HD44780, P12 CONN_BAT, P13 TP_GND, P14 TP_5V, P15 TP_3V, P16 TP_THERM_OUT, P17 TP_MULT_OUT, P18 TP_VREF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

Commit message: Fix Vss and Vdd swapped on display connector
Connections:
- net +5V: now also P11.2 (VDD); no longer P11.1 (VSS)
- net GND: now also P11.1 (VSS); no longer P11.2 (VDD)
Changed lines of the file:
@@
 L GND #PWR021
 U 1 1 57EBD86A
-P 950 6125
-F 0 "#PWR021" H 950 5875 50  0001 C CNN
-F 1 "GND" H 950 5975 50  0000 C CNN
-F 2 "" H 950 6125 50  0000 C CNN
-F 3 "" H 950 6125 50  0000 C CNN
-	1    950  6125
+P 1200 5800
+F 0 "#PWR021" H 1200 5550 50  0001 C CNN
+F 1 "GND" H 1200 5650 50  0000 C CNN
+F 2 "" H 1200 5800 50  0000 C CNN
+F 3 "" H 1200 5800 50  0000 C CNN
+	1    1200 5800
 	1    0    0    -1
 $EndComp
@@
 	2250 4300 2150 4300
 Wire Wire Line
-	950  6025 1400 6025
-Wire Wire Line
-	950  6125 1400 6125
-Wire Wire Line
 	950  7425 1400 7425
 Wire Wire Line
@@
 Wire Wire Line
 	9550 6025 9550 5900
+Wire Wire Line
+	1400 6025 1325 6025
+Wire Wire Line
+	1325 6025 1325 5725
+Wire Wire Line
+	1325 5725 1200 5725
+Wire Wire Line
+	1200 5725 1200 5800
+Wire Wire Line
+	1400 6125 950  6125
+Wire Wire Line
+	950  6125 950  6025
 $EndSCHEMATC
